File: hardware/electronics/PCBs/kicad/vertical_left/BigButtons.kicad_sch (KiCad schematic)
At the start: 2 parts, among them SW1 D2LS-21, SW2 D2LS-21

Commit message: add vertical
Parts:
- removed SW1, SW2: D2LS-21, D2LS-21, symbol Switches:LBS_0_D2LS-21_Switches.SchLib
- added SW1, SW2: D2LS-21, D2LS-21, symbol Switches:BBS_0_D2LS-21_Switches.SchLib
Connections:
- net GND: now also SW1.B, SW2.B
- new net ButtonLeftClick: SW1.A
- new net ButtonRightClick: SW2.A
Other:
- company: Ploopy Corporation -> (none)
