File: hardware/electronics/PCBs/kicad/vertical_left/ScrollWheel.kicad_sch (KiCad schematic)
At the start: 9 parts, among them SW3 D2LS-21

Commit message: Vertical portion flipped
Parts:
- removed R1: 0805, 0805, symbol Chip_Passives:SCW_1_Res 100R 1% 0805_Chip_Passives.SchLib
- added R1: 100, Resistor_SMD:R_0805_2012Metric, symbol Device:R_Small_US
- D1, D2: footprint IR12-21C/TR8 -> Library:TR8
- R2, R4: value 0805 -> 1k; footprint 0805 -> Resistor_SMD:R_0805_2012Metric
- R3: value 0805 -> 100; footprint 0805 -> Resistor_SMD:R_0805_2012Metric
Connections:
- net 3V3: now also Qt2.1 (C), R1.1; no longer Qt2.C
- net GND: now also D1.2 (C), D2.2 (C); no longer D1.C, D2.C
- net ScrollWheelOpto1: now also Qt2.2 (E); no longer Qt2.E
- net at R3.1: now also D2.1 (A); no longer D2.A
- new net: D1.1 (A), R1.2
- no-connect marks 1 -> 0
Other:
- moved on the sheet: Qt2
