File: hardware/electronics/PCBs/kicad/vertical_left/VerticalPCBConnection.kicad_sch (KiCad schematic)
At the start: 9 parts

Commit message: add vertical
Other:
- company: Ploopy Corporation -> (none)
