File: hardware/electronics/PCBs/kicad/vertical_left/Vertical.kicad_pcb (KiCad board)
At the start: 2 copper layers, 53.9 x 47.1 mm, 40 parts, among them SW1 D2LS-21, SW2 D2LS-21, SW3 D2LS-21

Commit message: Vertical neopixels
Parts:
- added C20: 100nF, Capacitor_SMD:C_0402_1005Metric, F.Cu at (179.1, 97.0)
- added C23: 100nF, Capacitor_SMD:C_0402_1005Metric, F.Cu at (179.1, 99.0)
- added C25: 100nF, Capacitor_SMD:C_0402_1005Metric, F.Cu at (179.1, 101.0)
- added CJ10: PCBJointCastellationJoint, PCBFeatures:PCBJoint, F.Cu at (130.0, 81.6)
- added CJ11: PCBJointCastellationJoint, PCBFeatures:PCBJoint, F.Cu at (170.0, 81.6)
- added R16: 1k, Resistor_SMD:R_0805_2012Metric, F.Cu at (182.7, 97.5)
- added R17: 1k, Resistor_SMD:R_0805_2012Metric, F.Cu at (182.7, 100.5)
- moved SW3 2.24 mm to (143.6, 98.5)
Routing:
- net /SCW/ButtonScrollWheel: track 26.2 -> 25.3 mm
- net GND: vias 42 -> 41

Commit message: PCB revs. Add vertical rgb leds. Fix sensor cutout
Parts:
- added D3: IN-PI55TATPRPGPB, LED_SMD:LED_WS2812B_PLCC4_5.0x5.0mm_P3.2mm, B.Cu at (128.7, 90.2)
- added D4: IN-PI55TATPRPGPB, LED_SMD:LED_WS2812B_PLCC4_5.0x5.0mm_P3.2mm, B.Cu at (169.4, 90.2)
- added D5: IN-PI55TATPRPGPB, LED_SMD:LED_WS2812B_PLCC4_5.0x5.0mm_P3.2mm, B.Cu at (128.7, 121.7)
- C20, C23, C25, R16, R17: moved to B.Cu
- moved R16 56.9 mm to (126.9, 86.2)
- moved C25 52.6 mm to (128.9, 116.7), turned to -135 degrees
- moved R17 51.8 mm to (136.6, 124.0)
- moved C20 48.4 mm to (131.8, 86.9)
- moved C23 14.3 mm to (171.9, 86.7)
- moved MCH.FID.2 3.42 mm to (169.4, 85.4)
- moved MCH.SP.9 1.49 mm to (172.9, 84.1)
Routing:
- net /LEDs/V_USB: track 0.00 -> 96.4 mm, vias 0 -> 4
- net Net-(D4-DOUT): track 0.00 -> 81.4 mm, vias 0 -> 2
- net Net-(D3-DOUT): track 0.00 -> 40.4 mm, vias 0 -> 2
- net Net-(D5-DOUT): track 0.00 -> 5.24 mm
- net /LEDs/LEDData: track 0.00 -> 4.80 mm
- net Net-(D3-DIN): track 0.00 -> 2.51 mm
- net Net-(D2-A): track 37.3 -> 39.4 mm
- net Net-(D1-A): track 47.6 -> 46.1 mm

Commit message: Correct IR footprints
Parts:
- D1, D2: footprint Library:TR8 -> IR:IR12-21CTR8
- Q1: renamed from Qt1; value PT26-51B/TR8 or PT12-21B/TR8 -> PT26-51B/TR8; footprint OptoElectronics:TR8 -> IR:PT26-51B-TR8
- Q2: renamed from Qt2; value PT26-51B/TR8 or PT12-21B/TR8 -> PT26-51B/TR8; footprint OptoElectronics:TR8 -> IR:PT26-51B-TR8
- turned D1 to 180 degrees
- turned D2 to 180 degrees
- turned Q1 to 0 degrees
- turned Q2 to 0 degrees
Connections:
- Q2 pad 1: /SCW/3V3 -> /SCW/ScrollWheelOpto1
- Q2 pad 2: /SCW/ScrollWheelOpto1 -> /SCW/3V3
Routing:
- net /SCW/ScrollWheelOpto0: track 44.3 -> 46.1 mm
- net /SCW/3V3: track 49.9 -> 48.7 mm
