File: hardware/electronics/PCBs/kicad/base2/LEDs.kicad_sch (KiCad schematic)
At the start: 8 parts

Commit message: add vertical
Parts:
- C20, C23, C25: footprint 0805 - TALL -> Capacitor_SMD:C_0805_2012Metric
- R16, R18: footprint 0805 -> Resistor_SMD:R_0805_2012Metric
Changed lines of the file:
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@@
 		(in_pos_files yes)
 		(dnp no)
-		(property "Reference" "#PWR?"
+		(property "Reference" "#PWR06"
 			(at 165.1 137.16 0)
 			(hide yes)
@@
 			(project "Base"
 				(path "/d0aa5c71-a42d-40bb-b9da-a8c48d59eca1/2ac03787-079d-4255-b19b-ad1352fc6cd6"
-					(reference "#PWR?")
+					(reference "#PWR06")
 					(unit 1)
 				)
@@
 			)
 		)
-		(property "Footprint" "0805 - TALL"
+		(property "Footprint" "Capacitor_SMD:C_0805_2012Metric"
 			(at 121.92 101.6 0)
 			(hide yes)
@@
 		(in_pos_files yes)
 		(dnp no)
-		(property "Reference" "#PWR?"
+		(property "Reference" "#PWR01"
 			(at 124.46 73.66 0)
 			(hide yes)
@@
 			(project "Base"
 				(path "/d0aa5c71-a42d-40bb-b9da-a8c48d59eca1/2ac03787-079d-4255-b19b-ad1352fc6cd6"
-					(reference "#PWR?")
+					(reference "#PWR01")
 					(unit 1)
 				)
@@
 		(in_pos_files yes)
 		(dnp no)
-		(property "Reference" "#PWR?"
+		(property "Reference" "#PWR05"
 			(at 165.1 106.68 0)
 			(hide yes)
@@
 			(project "Base"
 				(path "/d0aa5c71-a42d-40bb-b9da-a8c48d59eca1/2ac03787-079d-4255-b19b-ad1352fc6cd6"
-					(reference "#PWR?")
+					(reference "#PWR05")
 					(unit 1)
 				)
@@
 			)
 		)
-		(property "Footprint" "0805"
+		(property "Footprint" "Resistor_SMD:R_0805_2012Metric"
 			(at 129.54 147.32 0)
 			(hide yes)
@@
 			)
 		)
-		(property "Footprint" "0805 - TALL"
+		(property "Footprint" "Capacitor_SMD:C_0805_2012Metric"
 			(at 121.92 132.08 0)
 			(hide yes)
@@
 			)
 		)
-		(property "Footprint" "0805"
+		(property "Footprint" "Resistor_SMD:R_0805_2012Metric"
 			(at 160.02 55.88 0)
 			(hide yes)
@@
 			)
 		)
-		(property "Footprint" "0805 - TALL"
+		(property "Footprint" "Capacitor_SMD:C_0805_2012Metric"
 			(at 121.92 71.12 0)
 			(hide yes)
@@
 		(in_pos_files yes)
 		(dnp no)
-		(property "Reference" "#PWR?"
+		(property "Reference" "#PWR02"
 			(at 124.46 104.14 0)
 			(hide yes)
@@
 			(project "Base"
 				(path "/d0aa5c71-a42d-40bb-b9da-a8c48d59eca1/2ac03787-079d-4255-b19b-ad1352fc6cd6"
-					(reference "#PWR?")
+					(reference "#PWR02")
 					(unit 1)
 				)
@@
 		(in_pos_files yes)
 		(dnp no)
-		(property "Reference" "#PWR?"
+		(property "Reference" "#PWR04"
 			(at 165.1 76.2 0)
 			(hide yes)
@@
 			(project "Base"
 				(path "/d0aa5c71-a42d-40bb-b9da-a8c48d59eca1/2ac03787-079d-4255-b19b-ad1352fc6cd6"
-					(reference "#PWR?")
+					(reference "#PWR04")
 					(unit 1)
 				)
@@
 		(in_pos_files yes)
 		(dnp no)
-		(property "Reference" "#PWR?"
+		(property "Reference" "#PWR03"
 			(at 124.46 134.62 0)
 			(hide yes)
@@
 			(project "Base"
 				(path "/d0aa5c71-a42d-40bb-b9da-a8c48d59eca1/2ac03787-079d-4255-b19b-ad1352fc6cd6"
-					(reference "#PWR?")
+					(reference "#PWR03")
 					(unit 1)
 				)

Commit message: Getting parts right
Parts:
- C20, C23, C25: value 0805 -> 100nF; footprint Capacitor_SMD:C_0805_2012Metric -> Capacitor_SMD:C_0402_1005Metric
- R16, R18: value 0805 -> 1k
Changed lines of the file:
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@@
 			)
 		)
-		(property "Value" "0805"
+		(property "Value" "100nF"
 			(at 111.76 101.6 0)
 			(show_name no)
@@
 			)
 		)
-		(property "Footprint" "Capacitor_SMD:C_0805_2012Metric"
+		(property "Footprint" "Capacitor_SMD:C_0402_1005Metric"
 			(at 121.92 101.6 0)
 			(hide yes)
@@
 			)
 		)
-		(property "Value" "0805"
+		(property "Value" "1k"
 			(at 132.842 147.066 0)
 			(show_name no)
@@
 			)
 		)
-		(property "Value" "0805"
+		(property "Value" "100nF"
 			(at 111.76 132.08 0)
 			(show_name no)
@@
 			)
 		)
-		(property "Footprint" "Capacitor_SMD:C_0805_2012Metric"
+		(property "Footprint" "Capacitor_SMD:C_0402_1005Metric"
 			(at 121.92 132.08 0)
 			(hide yes)
@@
 			)
 		)
-		(property "Value" "0805"
+		(property "Value" "1k"
 			(at 154.686 56.642 90)
 			(show_name no)
@@
 			)
 		)
-		(property "Value" "0805"
+		(property "Value" "100nF"
 			(at 111.76 71.12 0)
 			(show_name no)
@@
 			)
 		)
-		(property "Footprint" "Capacitor_SMD:C_0805_2012Metric"
+		(property "Footprint" "Capacitor_SMD:C_0402_1005Metric"
 			(at 121.92 71.12 0)
 			(hide yes)
