File: hardware/electronics/PCBs/kicad/base2/MouseSensor.kicad_sch (KiCad schematic)
At the start: 6 parts, among them U2 PMW3360DM-T2QU

Commit message: add vertical
Parts:
- C10: value 0805 -> 10uF; footprint 0805 - TALL -> Capacitor_SMD:C_0805_2012Metric
- C11: value 0805 -> 100nF; footprint 0805 - TALL -> Capacitor_SMD:C_0805_2012Metric
- R3, R4: value 0805 -> 22R; footprint 0805 -> Resistor_SMD:R_0805_2012Metric
- R5: value 0805 -> 10k; footprint 0805 -> Resistor_SMD:R_0805_2012Metric
Connections:
- net MOSI: now also U2.11 (MOSI)
- net MOTION: now also U2.9 (MOTION)
- net SCLK: now also U2.10 (SCLK)
- net ~{CS}: now also U2.13 (~{CS})
- net ~{RESET}: now also U2.7 (~{RESET})
Changed lines of the file:
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@@
 	(hierarchical_label "~{CS}"
 		(shape input)
-		(at 175.26 91.44 180)
+		(at 160.02 91.44 0)
 		(effects
 			(font
 				(size 1.27 1.27)
 			)
-			(justify right)
+			(justify left)
 		)
 	)
 	(hierarchical_label "MOSI"
 		(shape input)
-		(at 175.26 99.06 180)
+		(at 160.02 99.06 0)
 		(effects
 			(font
 				(size 1.27 1.27)
 			)
-			(justify right)
+			(justify left)
 		)
 	)
 	(hierarchical_label "SCLK"
 		(shape input)
-		(at 175.26 101.6 180)
+		(at 160.02 101.6 0)
 		(effects
 			(font
 				(size 1.27 1.27)
 			)
-			(justify right)
+			(justify left)
 		)
 	)
@@
 	(hierarchical_label "~{RESET}"
 		(shape input)
-		(at 175.26 119.38 180)
+		(at 160.02 119.38 0)
 		(effects
 			(font
 				(size 1.27 1.27)
 			)
-			(justify right)
+			(justify left)
 		)
 	)
 	(hierarchical_label "MOTION"
 		(shape output)
-		(at 175.26 109.22 180)
+		(at 160.02 109.22 0)
 		(effects
 			(font
 				(size 1.27 1.27)
 			)
-			(justify right)
+			(justify left)
 		)
 	)
@@
 		(in_pos_files yes)
 		(dnp no)
-		(property "Reference" "#PWR?"
+		(property "Reference" "#PWR030"
 			(at 106.68 132.08 0)
 			(hide yes)
@@
 			(project "Base"
 				(path "/d0aa5c71-a42d-40bb-b9da-a8c48d59eca1/8a78d703-83b0-46e6-9d5c-1d446365bd9c"
-					(reference "#PWR?")
+					(reference "#PWR030")
 					(unit 1)
 				)
@@
 		(in_pos_files yes)
 		(dnp no)
-		(property "Reference" "#PWR?"
+		(property "Reference" "#PWR028"
 			(at 91.44 93.98 0)
 			(hide yes)
@@
 			(project "Base"
 				(path "/d0aa5c71-a42d-40bb-b9da-a8c48d59eca1/8a78d703-83b0-46e6-9d5c-1d446365bd9c"
-					(reference "#PWR?")
+					(reference "#PWR028")
 					(unit 1)
 				)
@@
 			)
 		)
-		(property "Value" "0805"
+		(property "Value" "10k"
 			(at 183.642 86.106 0)
 			(show_name no)
@@
 			)
 		)
-		(property "Footprint" "0805"
+		(property "Footprint" "Resistor_SMD:R_0805_2012Metric"
 			(at 180.34 86.36 0)
 			(hide yes)
@@
 			)
 		)
-		(property "Value" "0805"
+		(property "Value" "22R"
 			(at 163.322 81.026 0)
 			(show_name no)
@@
 			)
 		)
-		(property "Footprint" "0805"
+		(property "Footprint" "Resistor_SMD:R_0805_2012Metric"
 			(at 160.02 81.28 0)
 			(hide yes)
@@
 			)
 		)
-		(property "Value" "0805"
+		(property "Value" "10uF"
 			(at 93.726 93.726 0)
 			(show_name no)
@@
 			)
 		)
-		(property "Footprint" "0805 - TALL"
+		(property "Footprint" "Capacitor_SMD:C_0805_2012Metric"
 			(at 88.9 91.44 0)
 			(hide yes)
@@
 			)
 		)
-		(property "Value" "0805"
+		(property "Value" "100nF"
 			(at 108.966 93.726 0)
 			(show_name no)
@@
 			)
 		)
-		(property "Footprint" "0805 - TALL"
+		(property "Footprint" "Capacitor_SMD:C_0805_2012Metric"
 			(at 104.14 91.44 0)
 			(hide yes)
@@
 		(in_pos_files yes)
 		(dnp no)
-		(property "Reference" "#PWR?"
+		(property "Reference" "#PWR029"
 			(at 106.68 93.98 0)
 			(hide yes)
@@
 			(project "Base"
 				(path "/d0aa5c71-a42d-40bb-b9da-a8c48d59eca1/8a78d703-83b0-46e6-9d5c-1d446365bd9c"
-					(reference "#PWR?")
+					(reference "#PWR029")
 					(unit 1)
 				)
@@
 			)
 		)
-		(property "Value" "0805"
+		(property "Value" "22R"
 			(at 163.322 70.866 0)
 			(show_name no)
@@
 			)
 		)
-		(property "Footprint" "0805"
+		(property "Footprint" "Resistor_SMD:R_0805_2012Metric"
 			(at 160.02 71.12 0)
 			(hide yes)

Commit message: Getting parts right
Parts:
- C11: footprint Capacitor_SMD:C_0805_2012Metric -> Capacitor_SMD:C_0402_1005Metric
Connections:
- no-connect marks 3 -> 0
Changed lines of the file:
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@@
 		(color 0 0 0 0)
-	)
-	(no_connect
-		(at 116.84 109.22)
-	)
-	(no_connect
-		(at 160.02 86.36)
-	)
-	(no_connect
-		(at 116.84 116.84)
 	)
 	(wire
@@
 			)
 		)
-		(property "Footprint" "Capacitor_SMD:C_0805_2012Metric"
+		(property "Footprint" "Capacitor_SMD:C_0402_1005Metric"
 			(at 104.14 91.44 0)
 			(hide yes)
