File: hardware/electronics/PCBs/kicad/base2/Regulators.kicad_sch (KiCad schematic)
At the start: 8 parts, among them U3 AP2202K-3.3, U4 AP2204K-1.8

Commit message: add vertical
Parts:
- C12, C14, C16, C18: value 0805 -> 1uF; footprint 0805 - TALL -> Capacitor_SMD:C_0805_2012Metric
- C13, C17: value 0805 -> 10uF; footprint 0805 - TALL -> Capacitor_SMD:C_0805_2012Metric
Changed lines of the file:
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@@
 			)
 		)
-		(property "Value" "0805"
+		(property "Value" "1uF"
 			(at 177.546 75.946 0)
 			(show_name no)
@@
 			)
 		)
-		(property "Footprint" "0805 - TALL"
+		(property "Footprint" "Capacitor_SMD:C_0805_2012Metric"
 			(at 172.72 73.66 0)
 			(hide yes)
@@
 		(in_pos_files yes)
 		(dnp no)
-		(property "Reference" "#PWR?"
+		(property "Reference" "#PWR034"
 			(at 160.02 139.7 0)
 			(hide yes)
@@
 			(project "Base"
 				(path "/d0aa5c71-a42d-40bb-b9da-a8c48d59eca1/b93d6e5a-51c2-4578-bc1c-c9c8dffe719c"
-					(reference "#PWR?")
+					(reference "#PWR034")
 					(unit 1)
 				)
@@
 			)
 		)
-		(property "Value" "0805"
+		(property "Value" "1uF"
 			(at 177.546 139.446 0)
 			(show_name no)
@@
 			)
 		)
-		(property "Footprint" "0805 - TALL"
+		(property "Footprint" "Capacitor_SMD:C_0805_2012Metric"
 			(at 172.72 137.16 0)
 			(hide yes)
@@
 			)
 		)
-		(property "Value" "0805"
+		(property "Value" "10uF"
 			(at 162.306 139.446 0)
 			(show_name no)
@@
 			)
 		)
-		(property "Footprint" "0805 - TALL"
+		(property "Footprint" "Capacitor_SMD:C_0805_2012Metric"
 			(at 157.48 137.16 0)
 			(hide yes)
@@
 		(in_pos_files yes)
 		(dnp no)
-		(property "Reference" "#PWR?"
+		(property "Reference" "#PWR035"
 			(at 175.26 76.2 0)
 			(hide yes)
@@
 			(project "Base"
 				(path "/d0aa5c71-a42d-40bb-b9da-a8c48d59eca1/b93d6e5a-51c2-4578-bc1c-c9c8dffe719c"
-					(reference "#PWR?")
+					(reference "#PWR035")
 					(unit 1)
 				)
@@
 			)
 		)
-		(property "Value" "0805"
+		(property "Value" "1uF"
 			(at 101.346 139.446 0)
 			(show_name no)
@@
 			)
 		)
-		(property "Footprint" "0805 - TALL"
+		(property "Footprint" "Capacitor_SMD:C_0805_2012Metric"
 			(at 96.52 137.16 0)
 			(hide yes)
@@
 			)
 		)
-		(property "Value" "0805"
+		(property "Value" "10uF"
 			(at 162.306 75.946 0)
 			(show_name no)
@@
 			)
 		)
-		(property "Footprint" "0805 - TALL"
+		(property "Footprint" "Capacitor_SMD:C_0805_2012Metric"
 			(at 157.48 73.66 0)
 			(hide yes)
@@
 		(in_pos_files yes)
 		(dnp no)
-		(property "Reference" "#PWR?"
+		(property "Reference" "#PWR036"
 			(at 175.26 139.7 0)
 			(hide yes)
@@
 			(project "Base"
 				(path "/d0aa5c71-a42d-40bb-b9da-a8c48d59eca1/b93d6e5a-51c2-4578-bc1c-c9c8dffe719c"
-					(reference "#PWR?")
+					(reference "#PWR036")
 					(unit 1)
 				)
@@
 		(in_pos_files yes)
 		(dnp no)
-		(property "Reference" "#PWR?"
+		(property "Reference" "#PWR033"
 			(at 160.02 76.2 0)
 			(hide yes)
@@
 			(project "Base"
 				(path "/d0aa5c71-a42d-40bb-b9da-a8c48d59eca1/b93d6e5a-51c2-4578-bc1c-c9c8dffe719c"
-					(reference "#PWR?")
+					(reference "#PWR033")
 					(unit 1)
 				)
@@
 			)
 		)
-		(property "Value" "0805"
+		(property "Value" "1uF"
 			(at 101.346 75.946 0)
 			(show_name no)
@@
 			)
 		)
-		(property "Footprint" "0805 - TALL"
+		(property "Footprint" "Capacitor_SMD:C_0805_2012Metric"
 			(at 96.52 73.66 0)
 			(hide yes)
@@
 		(in_pos_files yes)
 		(dnp no)
-		(property "Reference" "#PWR?"
+		(property "Reference" "#PWR031"
 			(at 99.06 78.74 0)
 			(hide yes)
@@
 			(project "Base"
 				(path "/d0aa5c71-a42d-40bb-b9da-a8c48d59eca1/b93d6e5a-51c2-4578-bc1c-c9c8dffe719c"
-					(reference "#PWR?")
+					(reference "#PWR031")
 					(unit 1)
 				)
@@
 		(in_pos_files yes)
 		(dnp no)
-		(property "Reference" "#PWR?"
+		(property "Reference" "#PWR032"
 			(at 99.06 142.24 0)
 			(hide yes)
@@
 			(project "Base"
 				(path "/d0aa5c71-a42d-40bb-b9da-a8c48d59eca1/b93d6e5a-51c2-4578-bc1c-c9c8dffe719c"
-					(reference "#PWR?")
+					(reference "#PWR032")
 					(unit 1)
 				)

Commit message: Getting parts right
Parts:
- C12, C14, C16, C18: footprint Capacitor_SMD:C_0805_2012Metric -> Capacitor_SMD:C_0402_1005Metric
- U3: footprint AP2202 - SOT95P270X145-5N -> Package_TO_SOT_SMD:SOT-23-5
Changed lines of the file:
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@@
 			)
 		)
-		(property "Footprint" "Capacitor_SMD:C_0805_2012Metric"
+		(property "Footprint" "Capacitor_SMD:C_0402_1005Metric"
 			(at 172.72 73.66 0)
 			(hide yes)
@@
 			)
 		)
-		(property "Footprint" "AP2202 - SOT95P270X145-5N"
+		(property "Footprint" "Package_TO_SOT_SMD:SOT-23-5"
 			(at 124.46 73.66 0)
 			(hide yes)
@@
 			)
 		)
-		(property "Footprint" "Capacitor_SMD:C_0805_2012Metric"
+		(property "Footprint" "Capacitor_SMD:C_0402_1005Metric"
 			(at 172.72 137.16 0)
 			(hide yes)
@@
 			)
 		)
-		(property "Footprint" "Capacitor_SMD:C_0805_2012Metric"
+		(property "Footprint" "Capacitor_SMD:C_0402_1005Metric"
 			(at 96.52 137.16 0)
 			(hide yes)
@@
 			)
 		)
-		(property "Footprint" "Capacitor_SMD:C_0805_2012Metric"
+		(property "Footprint" "Capacitor_SMD:C_0402_1005Metric"
 			(at 96.52 73.66 0)
 			(hide yes)
