File: hardware/electronics/PCBs/kicad/base2/Base.kicad_pcb (KiCad board)
At the start: 4 copper layers, 79.4 x 68 mm, 72 parts

Commit message: add vertical
Parts:
- added C1: 100nF, Capacitor_SMD:C_0603_1608Metric, F.Cu at (218.2, 109.6)
- added C10: 10uF, Capacitor_SMD:C_0805_2012Metric, F.Cu at (220.7, 117.8)
- added C11: 100nF, Capacitor_SMD:C_0805_2012Metric, F.Cu at (220.7, 120.8)
- added C12: 1uF, Capacitor_SMD:C_0805_2012Metric, F.Cu at (192.7, 95.9)
- added C13: 10uF, Capacitor_SMD:C_0805_2012Metric, F.Cu at (198.9, 103.7)
- added C14: 1uF, Capacitor_SMD:C_0805_2012Metric, F.Cu at (198.9, 106.7)
- added C15: 100n, Capacitor_SMD:C_0402_1005Metric, F.Cu at (204.6, 104.1)
- added C16: 1uF, Capacitor_SMD:C_0805_2012Metric, F.Cu at (198.9, 109.7)
- added C17: 10uF, Capacitor_SMD:C_0805_2012Metric, F.Cu at (198.9, 112.7)
- added C18: 1uF, Capacitor_SMD:C_0805_2012Metric, F.Cu at (198.9, 115.7)
- added C20: 0805, Capacitor_SMD:C_0805_2012Metric, F.Cu at (205.4, 117.8)
- added C22: 4.7u, Capacitor_SMD:C_0402_1005Metric, F.Cu at (204.6, 106.0)
- added C23: 0805, Capacitor_SMD:C_0805_2012Metric, F.Cu at (205.4, 120.8)
- added C24: 100n, Capacitor_SMD:C_0402_1005Metric, F.Cu at (204.6, 108.0)
- added C25: 0805, Capacitor_SMD:C_0805_2012Metric, F.Cu at (205.4, 123.8)
- added C28: 4.7u, Capacitor_SMD:C_0402_1005Metric, F.Cu at (205.7, 97.0)
- added C29: 100n, Capacitor_SMD:C_0402_1005Metric, F.Cu at (207.5, 102.1)
- added C3: 15p, Capacitor_SMD:C_0402_1005Metric, F.Cu at (170.4, 106.4)
- added C30: 100n, Capacitor_SMD:C_0402_1005Metric, F.Cu at (207.5, 104.1)
- added C31: 100n, Capacitor_SMD:C_0402_1005Metric, F.Cu at (207.5, 106.0)
- added C32: 100n, Capacitor_SMD:C_0402_1005Metric, F.Cu at (207.5, 108.0)
- added C33: 100n, Capacitor_SMD:C_0402_1005Metric, F.Cu at (210.3, 100.1)
- added C34: 100n, Capacitor_SMD:C_0402_1005Metric, F.Cu at (210.3, 102.1)
- added C35: 100n, Capacitor_SMD:C_0402_1005Metric, F.Cu at (210.3, 104.1)
- added C4: 15p, Capacitor_SMD:C_0402_1005Metric, F.Cu at (204.6, 102.1)
- added R1: 0805, Resistor_SMD:R_0805_2012Metric, F.Cu at (214.0, 109.9)
- added R16: 0805, Resistor_SMD:R_0805_2012Metric, F.Cu at (209.8, 117.8)
- added R18: 0805, Resistor_SMD:R_0805_2012Metric, F.Cu at (209.8, 120.7)
- added R2: 0805, Resistor_SMD:R_0805_2012Metric, F.Cu at (214.0, 112.8)
- added R3: 22R, Resistor_SMD:R_0805_2012Metric, F.Cu at (216.2, 117.8)
- added R4: 22R, Resistor_SMD:R_0805_2012Metric, F.Cu at (216.2, 120.7)
- added R5: 10k, Resistor_SMD:R_0805_2012Metric, F.Cu at (216.2, 123.7)
- added R6: 33, Resistor_SMD:R_0402_1005Metric, F.Cu at (209.9, 110.0)
- added R7: 22R, Resistor_SMD:R_0805_2012Metric, F.Cu at (198.9, 120.7)
- added R8: 22R, Resistor_SMD:R_0805_2012Metric, F.Cu at (198.9, 123.6)
- added R9: 1k, Resistor_SMD:R_0402_1005Metric, F.Cu at (209.9, 112.0)
- added U6: RP2350A, Package_DFN_QFN:QFN-60-1EP_7x7mm_P0.4mm_EP3.4x3.4mm, F.Cu at (170.0, 98.4)
- added Y1: ABM8-272-T3, Crystal:Crystal_SMD_3225-4Pin_3.2x2.5mm, F.Cu at (167.6, 106.5)

Commit message: Getting parts right
Parts:
- removed the C10 at (220.7, 117.8)
- removed the C11 at (220.7, 120.8)
- removed the C16 at (198.9, 109.7)
- removed the C17 at (198.9, 112.7)
- removed the C18 at (198.9, 115.7)
- removed the C20 at (205.4, 117.8)
- removed the C23 at (205.4, 120.8)
- removed the C25 at (205.4, 123.8)
- removed the R16 at (209.8, 117.8)
- removed the R18 at (209.8, 120.7)
- removed the R3 at (216.2, 117.8)
- removed the R4 at (216.2, 120.7)
- removed the R7 at (198.9, 120.7)
- removed the R8 at (198.9, 123.6)
- removed USB.Ra.1: 1206 Quad, Chip_Passives:4x 10k 1% - CAC-80P320X160-8M
- added C26: 4.7uF, Capacitor_SMD:C_0402_1005Metric, F.Cu at (176.5, 98.4)
- added C27: 4.7uF, Capacitor_SMD:C_0402_1005Metric, F.Cu at (176.5, 95.9)
- added R10: 5.1k, Resistor_SMD:R_0402_1005Metric, F.Cu at (118.1, 95.2)
- added R11: 5.1k, Resistor_SMD:R_0402_1005Metric, F.Cu at (118.1, 97.2)
- added U1: W25Q16JVSSIQ, Package_SO:SOIC-8_5.3x6.2mm_P1.27mm, F.Cu at (167.6, 89.6)
- added U3: AP2202K-3.3, Package_TO_SOT_SMD:SOT-23-5, F.Cu at (169.7, 119.4)
- C1: footprint Capacitor_SMD:C_0603_1608Metric -> Capacitor_SMD:C_0402_1005Metric
- C10: renamed from MOS.C.10; value 0805 -> 10uF; footprint Chip_Passives:0805 - TALL -> Capacitor_SMD:C_0805_2012Metric
- C11: renamed from MOS.C.11; value 0805 -> 100nF; footprint Chip_Passives:0805 - TALL -> Capacitor_SMD:C_0402_1005Metric
- C12, C14: footprint Capacitor_SMD:C_0805_2012Metric -> Capacitor_SMD:C_0402_1005Metric
- C15, C24, C29, C30, C31, C32, C33, C34, C35: value 100n -> 100nF
- C16: renamed from REG.C.16; value 0805 -> 1uF; footprint Chip_Passives:0805 - TALL -> Capacitor_SMD:C_0402_1005Metric
- C17: renamed from REG.C.17; value 0805 -> 10uF; footprint Chip_Passives:0805 - TALL -> Capacitor_SMD:C_0805_2012Metric
- C18: renamed from REG.C.18; value 0805 -> 1uF; footprint Chip_Passives:0805 - TALL -> Capacitor_SMD:C_0402_1005Metric
- C20: renamed from LED.C.20; value 0805 -> 100nF; footprint Chip_Passives:0805 - TALL -> Capacitor_SMD:C_0402_1005Metric
- C22, C28: value 4.7u -> 4.7uF
- C23: renamed from LED.C.23; value 0805 -> 100nF; footprint Chip_Passives:0805 - TALL -> Capacitor_SMD:C_0402_1005Metric
- C25: renamed from LED.C.25; value 0805 -> 100nF; footprint Chip_Passives:0805 - TALL -> Capacitor_SMD:C_0402_1005Metric
- C3, C4: value 15p -> 15pF
- FB1: renamed from USB.FB.1; value ACML-0805-601-T -> GZ2012D601TF
- FB3: renamed from USB.FB.3; value ACML-0805-601-T -> GZ2012D601TF
- J3: renamed from USB.J.2; value DX07S016JA1R1500 -> C2760486; footprint Connectors:DX07S016JA1R1500 -> Adafruit:USB_C_Receptacle_HRO_TYPE-C-31-M-31
- R1: value 0805 -> 1k
- R16: renamed from LED.R.16; value 0805 -> 1k; footprint Chip_Passives:0805 -> Resistor_SMD:R_0805_2012Metric
- R18: renamed from LED.R.18; value 0805 -> 1k; footprint Chip_Passives:0805 -> Resistor_SMD:R_0805_2012Metric
- R2: value 0805 -> 10k
- R3: renamed from MOS.R.3; value 0805 -> 22R; footprint Chip_Passives:0805 -> Resistor_SMD:R_0805_2012Metric
- R4: renamed from MOS.R.4; value 0805 -> 22R; footprint Chip_Passives:0805 -> Resistor_SMD:R_0805_2012Metric
- R7: renamed from USB.R.7; value 0805 -> 22R; footprint Chip_Passives:0805 -> Resistor_SMD:R_0805_2012Metric
- R8: renamed from USB.R.8; value 0805 -> 22R; footprint Chip_Passives:0805 -> Resistor_SMD:R_0805_2012Metric
- moved R5 68.1 mm to (148.6, 116.2)
- moved R1 60.7 mm to (154.9, 123.8)
- moved C1 56.5 mm to (167.6, 84.5)
- moved R2 52.6 mm to (162.5, 123.8)
- moved R9 46.4 mm to (163.8, 106.1)
- moved C24 41.6 mm to (163.8, 99.7)
- moved C22 41.5 mm to (163.8, 98.4)
- moved C15 41.4 mm to (163.8, 97.2)
- moved C4 41.3 mm to (163.8, 108.6)
- moved R6 38.4 mm to (175.2, 93.4)
- moved C12 35.9 mm to (165.1, 118.8)
- moved C14 34.6 mm to (168.9, 123.8)
- moved C13 31.3 mm to (174.0, 122.6)
- moved C28 31.1 mm to (175.2, 90.8)
- moved C32 20.7 mm to (198.1, 89.6)
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- renumbered VPC.CJ.1 to CJ1, VPC.CJ.2 to CJ2, VPC.CJ.3 to CJ3, VPC.CJ.4 to CJ4, VPC.CJ.5 to CJ5, VPC.CJ.6 to CJ6, VPC.CJ.7 to CJ7, VPC.CJ.8 to CJ8, VPC.CJ.9 to CJ9, LED.D.1 to D1, LED.D.5 to D5, MCU.J.1 to J1, LBS.SW.1 to SW1, LBS.SW.2 to SW2, MOS.U.2 to U2, REG.U.4 to U4, USB.Z.1 to Z1
Connections:
- net NetLED.D.1_4 renamed Net-(D1-DIN)
- net NetLED.D.5_2 renamed Net-(D5-DOUT)
- net NetMOS.C.10_2 renamed Net-(U2-VDDPIX)
- net NetMOS.R.3_1 renamed Net-(R3-Pad1)
- net NetMOS.R.4_1 renamed Net-(U2-LED_P)
- net NetUSB.FB.3_2 renamed Net-(FB3-Pad2)
- C16 pad 2: V_USB -> /LED/V_USB
- C17 pad 2: 1V8 -> /MOS/1V8
- C18 pad 2: 1V8 -> /MOS/1V8
- C20 pad 2: V_USB -> /LED/V_USB
- C23 pad 2: V_USB -> /LED/V_USB
- C25 pad 2: V_USB -> /LED/V_USB
- CJ2 pad 1: NetMCU.U.5_32 -> /MCU/ButtonScrollWheel
- CJ3 pad 1: NetMCU.U.5_38 -> /MCU/ScrollWheelOpto0
- CJ4 pad 1: NetMCU.U.5_40 -> /MCU/ScrollWheelOpto1
- CJ6 pad 1: NetMCU.U.5_18 -> /MCU/ButtonLeftClick
- CJ7 pad 1: NetMCU.U.5_35 -> /MCU/ButtonRightClick
- CJ8 pad 1: 3V3 -> +3V3
- D1 pad 1: V_USB -> /LED/V_USB
- D1 pad 2: NetLED.D.1_2 -> Net-(D1-DOUT)
- D5 pad 1: V_USB -> /LED/V_USB
- D5 pad 4: NetLED.D.3_2 -> Net-(D3-DOUT)
- FB1 pad 1: NetUSB.FB.1_1 -> Net-(FB1-Pad1)
- FB1 pad 2: V_USB -> /LED/V_USB
- FB3 pad 1: NetUSB.FB.3_1 -> Net-(FB3-Pad1)
- R16 pad 2: LEDData -> /LED/LEDData
- R18 pad 1: (no net) -> unconnected-(R18-Pad1)
- R3 pad 2: 1V8 -> /MOS/1V8
- R7 pad 1: NetUSB.FB.2_2 -> Net-(FB2-Pad2)
- R7 pad 2: NetMCU.U.5_46 -> /MCU/D-
- R8 pad 2: NetMCU.U.5_47 -> /MCU/D+
- SW1 pad B: NetLBS.SW.1_B -> /LBS/ButtonRingFinger
- SW2 pad B: NetLBS.SW.2_B -> /LBS/ButtonLittleFinger
- U2 pad 1: (no net) -> unconnected-(U2-NC-Pad1)
- U2 pad 10: NetMCU.U.5_4 -> /MCU/SCLK
- U2 pad 11: NetMCU.U.5_9 -> /MCU/MOSI
- U2 pad 12: NetMCU.U.5_2 -> /MCU/MISO
- U2 pad 13: NetMCU.U.5_7 -> /MCU/~{CS}
- U2 pad 14: (no net) -> unconnected-(U2-NC-Pad14)
- U2 pad 16: (no net) -> unconnected-(U2-NC-Pad16)
- U2 pad 2: (no net) -> unconnected-(U2-NC-Pad2)
- U2 pad 4: 1V8 -> /MOS/1V8
- U2 pad 5: 3V3 -> +3V3
- U2 pad 6: (no net) -> unconnected-(U2-NC-Pad6)
- U2 pad 7: NetMCU.U.5_16 -> /MCU/~{RESET}
- U2 pad 9: NetMCU.U.5_12 -> /MCU/MOTION
- U4 pad 1: V_USB -> /LED/V_USB
- U4 pad 3: V_USB -> /LED/V_USB
- U4 pad 4: (no net) -> unconnected-(U4-NC-Pad4)
- U4 pad 5: 1V8 -> /MOS/1V8
- Z1 pad 1: NetUSB.FB.3_1 -> Net-(FB3-Pad1)
- Z1 pad 3: NetUSB.FB.2_1 -> Net-(FB2-Pad1)
- Z1 pad 4: NetUSB.FB.1_1 -> Net-(FB1-Pad1)
- Z1 pad 5: NetUSB.FB.1_1 -> Net-(FB1-Pad1)
- Z1 pad 6: (no net) -> unconnected-(Z1-Pad6)
Routing:
- net NetMCU.U.5_9: vias 2 -> 0
- net NetMCU.U.5_7: vias 1 -> 0
- net NetMCU.U.5_4: vias 3 -> 0
- net NetMCU.U.5_2: vias 1 -> 0
- net NetMCU.U.5_16: vias 1 -> 0
- net NetMCU.U.5_12: vias 1 -> 0
- net NetLED.D.1_2: vias 1 -> 0
- net NetLBS.SW.2_B: vias 1 -> 0
- net Net-(U2-VDDPIX): vias 0 -> 1
- net Net-(U1-~{HOLD}_or_~{RESET}_(IO3)): vias 0 -> 1
- net Net-(D1-DIN): vias 0 -> 1
- net GND: vias 180 -> 175
- net 3V3: vias 1 -> 0
- net /MCU/SCLK: vias 0 -> 1
- net /LED/V_USB: vias 0 -> 1
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- added copper zone on In1.Cu, net +3V3
- removed copper zone on In1.Cu, net 3V3

Commit message: To order
Parts:
- added J14: Conn_01x04, Connector_JST:JST_SH_BM04B-SRSS-TB_1x04-1MP_P1.00mm_Vertical, F.Cu at (182.6, 105.4)
- added L1: AOTA-B201610S3R3-101-T, RP2350_60QFN_minimal:L_pol_2016, F.Cu at (170.8, 107.4)
- C26, C27: footprint Capacitor_SMD:C_0402_1005Metric -> RP2350_60QFN_minimal:C_0402_1005Metric_small_pads
- FB2: renamed from USB.FB.2; value ACML-0805-601-T -> GZ2012D601TF
- J3: value C2760486 -> USB_C_Receptacle_USB2.0_16P
- R7, R8: value 22R -> 27; footprint Resistor_SMD:R_0805_2012Metric -> Resistor_SMD:R_0402_1005Metric
- U6: footprint Package_DFN_QFN:QFN-60-1EP_7x7mm_P0.4mm_EP3.4x3.4mm -> RP2350_60QFN_minimal:RP2350-QFN-60-1EP_7x7_P0.4mm_EP3.4x3.4mm_ThermalVias
- moved C29 47.6 mm to (166.5, 121.3), turned to 180 degrees
- moved C32 45.0 mm to (162.3, 116.8), turned to 180 degrees
- moved R8 42.6 mm to (167.5, 105.9)
- moved R7 41.8 mm to (168.6, 105.9)
- moved C33 36.8 mm to (174.2, 119.5)
- moved C31 36.6 mm to (163.2, 112.2), turned to 180 degrees
- moved C30 32.3 mm to (167.3, 108.1), turned to 90 degrees
- moved C35 30.7 mm to (175.1, 115.9)
- moved C34 30.7 mm to (174.0, 112.5)
- moved C17 28.5 mm to (132.5, 98.5), turned to 0 degrees
- moved C18 25.7 mm to (134.3, 100.1), turned to 0 degrees
- moved C16 25.4 mm to (131.1, 104.2), turned to 90 degrees
- moved U4 25.4 mm to (129.6, 101.3), turned to 180 degrees
- moved R2 24.3 mm to (155.8, 100.6), turned to -90 degrees
- moved C12 23.4 mm to (172.3, 96.5), turned to 180 degrees
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- renumbered LED.D.3 to D3
Connections:
- net +3V3 renamed +3.3V
- net Net-(FB3-Pad2) renamed /USB/USB_D+
- D3 pad 1: V_USB -> /LED/V_USB
- D3 pad 2: NetLED.D.3_2 -> Net-(D3-DOUT)
- D3 pad 4: NetLED.D.1_2 -> Net-(D1-DOUT)
- FB2 pad 1: NetUSB.FB.2_1 -> Net-(FB2-Pad1)
- FB2 pad 2: NetUSB.FB.2_2 -> /USB/USB_D-
- J1 pad 2: NetMCU.J.1_2 -> Net-(J1--)
- J3 pad A1: Net-(FB1-Pad1) -> GND
- J3 pad A12: (no net) -> GND
- J3 pad A4: unconnected-(J2-SBU2-Pad4) -> Net-(FB1-Pad1)
- J3 pad A5: GND -> Net-(J3-CC1)
- J3 pad A6: Net-(FB1-Pad1) -> Net-(FB3-Pad1)
- J3 pad A7: Net-(J2-CC1) -> Net-(FB2-Pad1)
- J3 pad A9: Net-(FB3-Pad1) -> Net-(FB1-Pad1)
- J3 pad B1: Net-(FB2-Pad1) -> GND
- J3 pad B12: (no net) -> GND
- J3 pad B4: Net-(J2-CC2) -> Net-(FB1-Pad1)
- J3 pad B5: GND -> Net-(J3-CC2)
- J3 pad B6: GND -> Net-(FB3-Pad1)
- J3 pad B7: Net-(FB3-Pad1) -> Net-(FB2-Pad1)
- J3 pad B8: Net-(FB2-Pad1) -> unconnected-(J3-SBU2-PadB8)
- J3 pad B9: GND -> Net-(FB1-Pad1)
- R1 pad 2: Net-(R1-Pad2) -> /MCU/CS
- R2 pad 2: Net-(R1-Pad2) -> /MCU/CS
- R7 pad 1: Net-(FB2-Pad2) -> /USB/USB_D-
- U6 pad 12: GND -> unconnected-(U6-GPIO8-Pad12)
- U6 pad 14: GND -> unconnected-(U6-GPIO10-Pad14)
- U6 pad 15: GND -> unconnected-(U6-GPIO11-Pad15)
- U6 pad 18: GND -> unconnected-(U6-GPIO14-Pad18)
- U6 pad 27: GND -> unconnected-(U6-GPIO16-Pad27)
- U6 pad 29: GND -> unconnected-(U6-GPIO18-Pad29)
- U6 pad 3: GND -> unconnected-(U6-GPIO1-Pad3)
- U6 pad 32: GND -> unconnected-(U6-GPIO20-Pad32)
- U6 pad 34: GND -> /SDA
- U6 pad 35: /MCU/ButtonRightClick -> /SCL
- U6 pad 36: GND -> /MCU/ButtonRightClick
- U6 pad 37: GND -> unconnected-(U6-GPIO25-Pad37)
- U6 pad 41: GND -> unconnected-(U6-GPIO27/ADC1-Pad41)
- U6 pad 43: GND -> unconnected-(U6-GPIO29/ADC3-Pad43)
- U6 pad 5: GND -> unconnected-(U6-GPIO3-Pad5)
- U6 pad 7: GND -> unconnected-(U6-GPIO4-Pad7)
- U6 pad 9: GND -> unconnected-(U6-GPIO6-Pad9)
Routing:
- net /LED/V_USB: track 0.00 -> 142.3 mm, vias 1 -> 6
- net +3.3V: track 0.00 -> 111.4 mm, vias 0 -> 3
- net /MCU/ButtonScrollWheel: track 0.00 -> 83.0 mm, vias 0 -> 3
- net /MCU/ScrollWheelOpto0: track 0.00 -> 66.2 mm, vias 0 -> 1
- net /USB/USB_D-: track 0.00 -> 62.0 mm
- net /USB/USB_D+: track 0.00 -> 61.3 mm
- net /MCU/ScrollWheelOpto1: track 0.00 -> 60.5 mm, vias 0 -> 1
- net /MCU/ButtonLeftClick: track 0.00 -> 59.6 mm, vias 0 -> 6
- net Net-(D1-DOUT): track 0.00 -> 54.9 mm
- net /MCU/ButtonRightClick: track 0.00 -> 54.7 mm, vias 0 -> 1
- net Net-(D3-DOUT): track 0.00 -> 47.0 mm
- net /MOS/1V8: track 0.00 -> 41.0 mm, vias 0 -> 1
- net /LED/LEDData: track 0.00 -> 38.2 mm, vias 1 -> 4
- net /LBS/ButtonRingFinger: track 0.00 -> 36.0 mm
- net /MCU/~{RESET}: track 0.00 -> 32.3 mm, vias 0 -> 4
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- added copper zone on F.Cu, net +1V1
- added copper zone on F.Cu, net +3.3V
- removed copper zone on In1.Cu, net +3.3V
- removed copper zone on In1.Cu, net GND
- removed copper zone on In2.Cu, net GND
Other:
- copper layers 4 -> 2
- rule pad_to_mask_clearance: 0.0762 -> 0
- board text added: "Nothing up here"
