File: hardware/electronics/PCBs/kicad/base2/Base.kicad_sch (KiCad schematic)
At the start: 0 parts

Commit message: To order
Parts:
- added J14: Conn_01x04, Connector_JST:JST_SH_BM04B-SRSS-TB_1x04-1MP_P1.00mm_Vertical, symbol Connector_Generic:Conn_01x04
Connections:
- new net +3.3V: J14.2 (Pin_2)
- new net GND: J14.1 (Pin_1)
- new net SCL: J14.4 (Pin_4)
- new net SDA: J14.3 (Pin_3)
Other:
- sheet MCU ports: added SCL, SDA; removed none
