File: hardware/electronics/PCBs/kicad/base2/Base.kicad_sch (KiCad schematic)
At the start: 1 part, among them J14 Conn_01x04

Commit message: Vertical neopixels
Other:
- sheet LED ports: added LEDDataOut; removed none
- sheet VPC ports: added 5V, LEDDataOut; removed none
Changed lines of the file:
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@@
+	)
+	(junction
+		(at 91.44 71.12)
+		(diameter 0)
+		(color 0 0 0 0)
 	)
 	(junction
@@
 	(wire
 		(pts
+			(xy 124.46 50.8) (xy 83.82 50.8)
+		)
+		(stroke
+			(width 0)
+			(type default)
+		)
+	)
+	(wire
+		(pts
+			(xy 81.28 71.12) (xy 81.28 109.22)
+		)
+		(stroke
+			(width 0)
+			(type default)
+		)
+	)
+	(wire
+		(pts
 			(xy 91.44 83.82) (xy 139.7 83.82)
 		)
@@
 	(wire
 		(pts
+			(xy 83.82 114.3) (xy 96.52 114.3)
+		)
+		(stroke
+			(width 0)
+			(type default)
+		)
+	)
+	(wire
+		(pts
+			(xy 81.28 109.22) (xy 96.52 109.22)
+		)
+		(stroke
+			(width 0)
+			(type default)
+		)
+	)
+	(wire
+		(pts
 			(xy 93.98 106.68) (xy 91.44 106.68)
 		)
@@
 	(wire
 		(pts
+			(xy 83.82 50.8) (xy 83.82 114.3)
+		)
+		(stroke
+			(width 0)
+			(type default)
+		)
+	)
+	(wire
+		(pts
 			(xy 91.44 60.96) (xy 91.44 71.12)
 		)
@@
 	(wire
 		(pts
+			(xy 124.46 58.42) (xy 124.46 50.8)
+		)
+		(stroke
+			(width 0)
+			(type default)
+		)
+	)
+	(wire
+		(pts
 			(xy 91.44 83.82) (xy 91.44 78.74)
+		)
+		(stroke
+			(width 0)
+			(type default)
+		)
+	)
+	(wire
+		(pts
+			(xy 91.44 71.12) (xy 81.28 71.12)
 		)
 		(stroke
@@
 			)
 		)
+		(pin "LEDDataOut" input
+			(at 124.46 58.42 90)
+			(effects
+				(font
+					(size 1.27 1.27)
+				)
+				(justify right)
+			)
+		)
 		(instances
 			(project "Base"
@@
 			)
 		)
+		(pin "LEDDataOut" input
+			(at 96.52 114.3 180)
+			(effects
+				(font
+					(size 1.27 1.27)
+				)
+				(justify left)
+			)
+		)
+		(pin "5V" input
+			(at 96.52 109.22 180)
+			(effects
+				(font
+					(size 1.27 1.27)
+				)
+				(justify left)
+			)
+		)
