File: hardware/electronics/PCBs/kicad/base2/MCU.kicad_sch (KiCad schematic)
At the start: 18 parts, among them J1 HEADER2, U1 W25Q16JVSSIQ, U5 RP2040, Y1 RH100-12.000-16-3030

Commit message: add vertical
Parts:
- removed C19, C21, C3, C4, C5, C6, C7, C8: 0603 X5R, 0603 capacitor - CAPC1608X06N, symbol Chip_Passives:MCU_1_Cap 0.1uF 25V_Chip_Passives.SchLib
- removed C2, C9: 0805 X5R, 0805 - TALL, symbol Chip_Passives:MCU_1_Cap 1uF 25V_Chip_Passives.SchLib
- removed R6: 0805, 0805, symbol Chip_Passives:MCU_2_Res 1k 1% 0805_Chip_Passives.SchLib
- removed U5: RP2040, RP2040 - QFN40P700X700X90_HS-57M, symbol MCUs:MCU_0_RP2040_MCUs.SchLib
- removed Y1: RH100-12.000-16-3030, RH100-12.000-16-3030, symbol Crystals:MCU_0_RH100-12.000-16-3030_Crystals.SchLib
- added C15, C24, C29, C30, C31, C32, C33, C34, C35: 100n, Capacitor_SMD:C_0402_1005Metric, symbol Device:C
- added C22, C28: 4.7u, Capacitor_SMD:C_0402_1005Metric, symbol Device:C
- added C26, C27: 4.7u, RP2350_60QFN_minimal:C_0402_1005Metric_small_pads, symbol Device:C
- added C3, C4: 15p, Capacitor_SMD:C_0402_1005Metric, symbol Device:C
- added L1: 3.3u, RP2350_60QFN_minimal:L_pol_2016, symbol Device:L
- added R6: 33, Resistor_SMD:R_0402_1005Metric, symbol Device:R
- added R9: 1k, Resistor_SMD:R_0402_1005Metric, symbol Device:R
- added U6: RP2350A, Package_DFN_QFN:QFN-60-1EP_7x7mm_P0.4mm_EP3.4x3.4mm, symbol MCU_RaspberryPi:RP2350A
- added Y1: ABM8-272-T3, Crystal:Crystal_SMD_3225-4Pin_3.2x2.5mm, symbol Device:Crystal_GND24
- C1: value 0603 X5R -> 100nF; footprint 0603 capacitor - CAPC1608X06N -> Capacitor_SMD:C_0603_1608Metric
- R1, R2: footprint 0805 -> Resistor_SMD:R_0805_2012Metric
Connections:
- net ButtonLeftClick: now also U6.19 (GPIO15)
- net ButtonLittleFinger: now also U6.31 (GPIO19)
- net ButtonRightClick: now also U6.35 (GPIO23)
- net ButtonRingFinger: now also U6.28 (GPIO17)
- net ButtonScrollWheel: now also U6.33 (GPIO21)
- net D+: now also U6.52 (USB_DP)
- net D-: now also U6.51 (USB_DM)
- net GND: now also C15.2, C22.2, C24.2, C26.2, C27.2, C28.2, C29.2, C3.2, C30.2, C31.2, C32.2, C33.2, C34.2, C35.2, C4.2, U6.12 (GPIO8), U6.14 (GPIO10), U6.15 (GPIO11), U6.18 (GPIO14), U6.27 (GPIO16), U6.29 (GPIO18), U6.3 (GPIO1), U6.32 (GPIO20), U6.34 (GPIO22), U6.36 (GPIO24), U6.37 (GPIO25), U6.41 (GPIO27/ADC1), U6.43 (GPIO29/ADC3), U6.47 (VREG_PGND), U6.5 (GPIO3), U6.61 (GND), U6.7 (GPIO4), U6.9 (GPIO6), Y1.2, Y1.4
- net LEDData: now also U6.16 (GPIO12)
- net MISO: now also U6.2 (GPIO0)
- net MOSI: now also U6.10 (GPIO7)
- net MOTION: now also U6.13 (GPIO9)
- net SCLK: now also U6.4 (GPIO2)
- net ScrollWheelOpto0: now also U6.40 (GPIO26/ADC0)
- net ScrollWheelOpto1: now also U6.42 (GPIO28/ADC2)
- net ~{CS}: now also U6.8 (GPIO5)
- net ~{RESET}: now also U6.17 (GPIO13)
- net at R1.2, R2.2: no longer U1.1 (~{CS})
- net at U1.2 (DO_(IO1)): now also U6.59 (QSPI_SD1)
- net at U1.3 (~{WP}_(IO2)): now also U6.58 (QSPI_SD2)
- net at U1.5 (DI_(IO0)): now also U6.57 (QSPI_SD0)
- net at U1.6 (CLK): now also U6.56 (QSPI_SCLK)
- net at U1.7 (~{HOLD}_or_~{RESET}_(IO3)): now also U6.55 (QSPI_SD3)
- net 3V3 renamed +3V3
- net +3V3: now also C26.1, C29.1, C30.1, C31.1, C32.1, C33.1, C34.1, C35.1, R6.1, U6.1 (IOVDD), U6.11 (IOVDD), U6.20 (IOVDD), U6.26 (RUN), U6.30 (IOVDD), U6.38 (IOVDD), U6.44 (ADC_AVDD), U6.45 (IOVDD), U6.49 (VREG_VIN), U6.53 (USB_OTP_VDD), U6.54 (QSPI_IOVDD)
- new net: C4.1, R9.2, Y1.3
- new net +1V1: C15.1, C22.1, C24.1, C27.1, L1.1, U6.23 (DVDD), U6.39 (DVDD), U6.50 (VREG_FB), U6.6 (DVDD)
- new net CS: U1.1 (~{CS}), U6.60 (~{QSPI_SS})
- new net VREG_AVDD: C28.1, R6.2, U6.46 (VREG_AVDD)
- new net VREG_LX: L1.2, U6.48 (VREG_LX)
- new net XIN: C3.1, U6.21 (XIN), Y1.1
- new net XOUT: R9.1, U6.22 (XOUT)
- no-connect marks 19 -> 2
Other:
- note added: "12MHz Crystal"
- moved on the sheet: C1, U1

Commit message: Getting parts right
Parts:
- C1: footprint Capacitor_SMD:C_0603_1608Metric -> Capacitor_SMD:C_0402_1005Metric
- C15, C24, C29, C30, C31, C32, C33, C34, C35: value 100n -> 100nF
- C22, C28: value 4.7u -> 4.7uF
- C26, C27: value 4.7u -> 4.7uF; footprint RP2350_60QFN_minimal:C_0402_1005Metric_small_pads -> Capacitor_SMD:C_0402_1005Metric
- C3, C4: value 15p -> 15pF
- L1: value 3.3u -> 3.3uH
- R1: value 0805 -> 1k
- R2: value 0805 -> 10k
- U1: footprint W25Q128JVS - SOIC127P790X216-8M -> Package_SO:SOIC-8_5.3x6.2mm_P1.27mm
Changed lines of the file:
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@@
 			)
 		)
-		(property "Footprint" "W25Q128JVS - SOIC127P790X216-8M"
+		(property "Footprint" "Package_SO:SOIC-8_5.3x6.2mm_P1.27mm"
 			(at 144.78 184.15 0)
 			(hide yes)
@@
 			)
 		)
-		(property "Value" "100n"
+		(property "Value" "100nF"
 			(at 70.231 124.333 0)
 			(show_name no)
@@
 			)
 		)
-		(property "Value" "15p"
+		(property "Value" "15pF"
 			(at 138.557 226.441 0)
 			(show_name no)
@@
 			)
 		)
-		(property "Value" "100n"
+		(property "Value" "100nF"
 			(at 159.258 111.76 0)
 			(show_name no)
@@
 			)
 		)
-		(property "Value" "0805"
+		(property "Value" "10k"
 			(at 225.806 84.4042 90)
 			(show_name no)
@@
 			)
 		)
-		(property "Value" "100n"
+		(property "Value" "100nF"
 			(at 124.841 111.633 0)
 			(show_name no)
@@
 		(fields_autoplaced yes)
 		(property "Reference" "C27"
-			(at 60.96 96.52 0)
+			(at 60.96 96.5199 0)
 			(show_name no)
 			(do_not_autoplace no)
@@
 			)
 		)
-		(property "Value" "4.7u"
-			(at 60.96 99.06 0)
+		(property "Value" "4.7uF"
+			(at 60.96 99.0599 0)
 			(show_name no)
 			(do_not_autoplace no)
@@
 			)
 		)
-		(property "Footprint" "RP2350_60QFN_minimal:C_0402_1005Metric_small_pads"
+		(property "Footprint" "Capacitor_SMD:C_0402_1005Metric"
 			(at 58.1152 101.6 0)
 			(hide yes)
@@
 			)
 		)
-		(property "Value" "15p"
+		(property "Value" "15pF"
 			(at 138.557 236.601 0)
 			(show_name no)
@@
 		(fields_autoplaced yes)
 		(property "Reference" "C28"
-			(at 95.25 83.82 0)
+			(at 95.25 83.8199 0)
 			(show_name no)
 			(do_not_autoplace no)
@@
 			)
 		)
-		(property "Value" "4.7u"
-			(at 95.25 86.36 0)
+		(property "Value" "4.7uF"
+			(at 95.25 86.3599 0)
 			(show_name no)
 			(do_not_autoplace no)
@@
 			)
 		)
-		(property "Value" "100n"
+		(property "Value" "100nF"
 			(at 181.991 111.633 0)
 			(show_name no)
@@
 			)
 		)
-		(property "Value" "4.7u"
+		(property "Value" "4.7uF"
 			(at 58.801 124.333 0)
 			(show_name no)
@@
 			)
 		)
-		(property "Value" "100n"
+		(property "Value" "100nF"
 			(at 47.371 124.333 0)
 			(show_name no)
@@
 			)
 		)
-		(property "Value" "100n"
+		(property "Value" "100nF"
 			(at 113.411 111.633 0)
 			(show_name no)
@@
 			)
 		)
-		(property "Value" "100n"
+		(property "Value" "100nF"
 			(at 147.701 111.633 0)
 			(show_name no)
@@
 		(fields_autoplaced yes)
 		(property "Reference" "L1"
-			(at 73.66 96.52 0)
+			(at 73.66 96.5199 0)
 			(show_name no)
 			(do_not_autoplace no)
@@
 			)
 		)
-		(property "Value" "3.3u"
-			(at 73.66 99.06 0)
+		(property "Value" "3.3uH"
+			(at 73.66 99.0599 0)
 			(show_name no)
 			(do_not_autoplace no)
@@
 			)
 		)
-		(property "Value" "0805"
+		(property "Value" "1k"
 			(at 200.406 84.4042 90)
 			(show_name no)
@@
 			)
 		)
-		(property "Value" "100n"
+		(property "Value" "100nF"
 			(at 170.561 111.633 0)
 			(show_name no)
@@
 			)
 		)
-		(property "Value" "100n"
+		(property "Value" "100nF"
 			(at 136.271 111.633 0)
 			(show_name no)
@@
 			)
 		)
-		(property "Footprint" "Capacitor_SMD:C_0603_1608Metric"
+		(property "Footprint" "Capacitor_SMD:C_0402_1005Metric"
 			(at 177.8 181.61 0)
 			(hide yes)
@@
 		(fields_autoplaced yes)
 		(property "Reference" "C26"
-			(at 48.641 96.9553 0)
+			(at 49.53 96.5199 0)
 			(show_name no)
 			(do_not_autoplace no)
@@
 			)
 		)
-		(property "Value" "4.7u"
-			(at 48.641 99.4922 0)
+		(property "Value" "4.7uF"
+			(at 49.53 99.0599 0)
 			(show_name no)
 			(do_not_autoplace no)
@@
 			)
 		)
-		(property "Footprint" "RP2350_60QFN_minimal:C_0402_1005Metric_small_pads"
+		(property "Footprint" "Capacitor_SMD:C_0402_1005Metric"
 			(at 46.6852 101.6 0)
 			(hide yes)

Commit message: To order
Parts:
- C26, C27: footprint Capacitor_SMD:C_0402_1005Metric -> RP2350_60QFN_minimal:C_0402_1005Metric_small_pads
- L1: value 3.3uH -> AOTA-B201610S3R3-101-T
- U6: footprint Package_DFN_QFN:QFN-60-1EP_7x7mm_P0.4mm_EP3.4x3.4mm -> RP2350_60QFN_minimal:RP2350-QFN-60-1EP_7x7_P0.4mm_EP3.4x3.4mm_ThermalVias
Connections:
- net ButtonRightClick: now also U6.36 (GPIO24); no longer U6.35 (GPIO23)
- net CS: now also R1.2, R2.2
- net GND: no longer U6.12 (GPIO8), U6.14 (GPIO10), U6.15 (GPIO11), U6.18 (GPIO14), U6.27 (GPIO16), U6.29 (GPIO18), U6.3 (GPIO1), U6.32 (GPIO20), U6.34 (GPIO22), U6.36 (GPIO24), U6.37 (GPIO25), U6.41 (GPIO27/ADC1), U6.43 (GPIO29/ADC3), U6.5 (GPIO3), U6.7 (GPIO4), U6.9 (GPIO6)
- new net SCL: U6.35 (GPIO23)
- new net SDA: U6.34 (GPIO22)
