File: hardware/electronics/PCBs/kicad/base2/USB.kicad_sch (KiCad schematic)
At the start: 8 parts, among them J2 DX07S016JA1R1500

Commit message: add vertical
Parts:
- R7, R8: value 0805 -> 22R; footprint 0805 -> Resistor_SMD:R_0805_2012Metric
- Ra1: value 1206 Quad -> 10k
Changed lines of the file:
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@@
 		(in_pos_files yes)
 		(dnp no)
-		(property "Reference" "#PWR?"
+		(property "Reference" "#PWR039"
 			(at 121.92 109.22 0)
 			(hide yes)
@@
 			(project "Base"
 				(path "/d0aa5c71-a42d-40bb-b9da-a8c48d59eca1/66301f0c-b18a-4a4e-81f3-7fe51cd45b0d"
-					(reference "#PWR?")
+					(reference "#PWR039")
 					(unit 1)
 				)
@@
 			)
 		)
-		(property "Value" "1206 Quad"
+		(property "Value" "10k"
 			(at 76.962 103.886 0)
 			(show_name no)
@@
 			)
 		)
-		(property "Value" "1206 Quad"
+		(property "Value" "10k"
 			(at 130.302 103.886 0)
 			(show_name no)
@@
 		(in_pos_files yes)
 		(dnp no)
-		(property "Reference" "#PWR?"
+		(property "Reference" "#PWR037"
 			(at 58.42 114.3 0)
 			(hide yes)
@@
 			(project "Base"
 				(path "/d0aa5c71-a42d-40bb-b9da-a8c48d59eca1/66301f0c-b18a-4a4e-81f3-7fe51cd45b0d"
-					(reference "#PWR?")
+					(reference "#PWR037")
 					(unit 1)
 				)
@@
 		(in_pos_files yes)
 		(dnp no)
-		(property "Reference" "#PWR?"
+		(property "Reference" "#PWR040"
 			(at 157.48 144.78 0)
 			(hide yes)
@@
 			(project "Base"
 				(path "/d0aa5c71-a42d-40bb-b9da-a8c48d59eca1/66301f0c-b18a-4a4e-81f3-7fe51cd45b0d"
-					(reference "#PWR?")
+					(reference "#PWR040")
 					(unit 1)
 				)
@@
 		(in_pos_files yes)
 		(dnp no)
-		(property "Reference" "#PWR?"
+		(property "Reference" "#PWR038"
 			(at 81.28 109.22 0)
 			(hide yes)
@@
 			(project "Base"
 				(path "/d0aa5c71-a42d-40bb-b9da-a8c48d59eca1/66301f0c-b18a-4a4e-81f3-7fe51cd45b0d"
-					(reference "#PWR?")
+					(reference "#PWR038")
 					(unit 1)
 				)
@@
 			)
 		)
-		(property "Value" "0805"
+		(property "Value" "22R"
 			(at 238.506 94.742 90)
 			(show_name no)
@@
 			)
 		)
-		(property "Footprint" "0805"
+		(property "Footprint" "Resistor_SMD:R_0805_2012Metric"
 			(at 238.76 88.9 0)
 			(hide yes)
@@
 			)
 		)
-		(property "Value" "0805"
+		(property "Value" "22R"
 			(at 238.506 104.902 90)
 			(show_name no)
@@
 			)
 		)
-		(property "Footprint" "0805"
+		(property "Footprint" "Resistor_SMD:R_0805_2012Metric"
 			(at 238.76 99.06 0)
 			(hide yes)
@@
 			)
 		)
-		(property "Value" "1206 Quad"
+		(property "Value" "10k"
 			(at 92.202 103.886 0)
 			(show_name no)
@@
 			)
 		)
-		(property "Value" "1206 Quad"
+		(property "Value" "10k"
 			(at 115.062 103.886 0)
 			(show_name no)

Commit message: Getting parts right
Parts:
- removed J2: DX07S016JA1R1500, DX07S016JA1R1500, symbol Connectors:USB_0_mirrored_DX07S016JA1R1500_Connectors.SchLib
- removed Ra1: 10k, 4x 10k 1% - CAC-80P320X160-8M, symbol Chip_Passives:USB_1_Quad Res 10k 1% 1206_Chip_Passives.SchLib
- added J3: USB_C_Receptacle_USB2.0_16P, Adafruit:USB_C_Receptacle_HRO_TYPE-C-31-M-31, symbol Connector:USB_C_Receptacle_USB2.0_16P
- added R10, R11: 5.1k, Resistor_SMD:R_0402_1005Metric, symbol Device:R_Small_US
- FB1, FB2, FB3: value ACML-0805-601-T -> GZ2012D601TF
Connections:
- net GND: now also J3.A1 (GND), J3.A12 (GND), J3.B1 (GND), J3.B12 (GND), J3.SH (SHIELD), R10.2, R11.2
- net at FB3.1, Z1.1: now also J3.A6 (D+), J3.B6 (D+)
- net at FB2.1, Z1.3: now also J3.A7 (D-), J3.B7 (D-)
- net at FB1.1, Z1.4, Z1.5: now also J3.A4 (VBUS), J3.A9 (VBUS), J3.B4 (VBUS), J3.B9 (VBUS)
- new net: J3.A5 (CC1), R10.1
- new net: J3.B5 (CC2), R11.1
- no-connect marks 0 -> 2

Commit message: To order
Parts:
- R7, R8: value 22R -> 27; footprint Resistor_SMD:R_0805_2012Metric -> Resistor_SMD:R_0402_1005Metric
Connections:
- net USB_D+: now reaches FB3.2, R8.1
- net USB_D-: now reaches FB2.2, R7.1
Changed lines of the file:
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@@
+		)
+	)
+	(label "USB_D-"
+		(at 217.17 91.44 0)
+		(effects
+			(font
+				(size 1.27 1.27)
+			)
+			(justify left bottom)
+		)
+	)
+	(label "USB_D+"
+		(at 217.17 101.6 0)
+		(effects
+			(font
+				(size 1.27 1.27)
+			)
+			(justify left bottom)
 		)
 	)
@@
 			)
 		)
-		(property "Value" "22R"
+		(property "Value" "27"
 			(at 238.506 94.742 90)
 			(show_name no)
@@
 			)
 		)
-		(property "Footprint" "Resistor_SMD:R_0805_2012Metric"
+		(property "Footprint" "Resistor_SMD:R_0402_1005Metric"
 			(at 238.76 88.9 0)
 			(hide yes)
@@
 			)
 		)
-		(property "Value" "22R"
+		(property "Value" "27"
 			(at 238.506 104.902 90)
 			(show_name no)
@@
 			)
 		)
-		(property "Footprint" "Resistor_SMD:R_0805_2012Metric"
+		(property "Footprint" "Resistor_SMD:R_0402_1005Metric"
 			(at 238.76 99.06 0)
 			(hide yes)
